File: USB-DMX FT232.kicad_pcb (KiCad board)
At the start: 2 copper layers, 66.7 x 29 mm, 26 parts, among them J1 USB, J2 NC3MAFH-PH, U1 FT232RL, U2 TEA1-0505, U3 6N137, U4 MAX485E

Commit message: usbc version
Parts:
- removed J1: USB, Connector_USB:USB_B_Lumberg_2411_02_Horizontal
- added P1: USB_C_Plug_USB2.0, Connector_USB:USB_C_Receptacle_JAE_DX07S016JA1R1500, F.Cu at (94.1, 85.1)
- added R9: 5.1k, Resistor_SMD:R_0805_2012Metric_Pad1.20x1.40mm_HandSolder, F.Cu at (100.6, 81.8)
- J2: footprint UncleEugeneParts:XLR 3pin Female Angle -> Uncleeugene:XLR 3pin Female Angle
Routing:
- net VCC: track 70.6 -> 78.7 mm, vias 2 -> 4
- net GND: track 3.39 -> 9.95 mm
- net Net-(P1-CC): track 0.00 -> 4.17 mm
- net Net-(P1-D+): track 15.3 -> 12.2 mm
- net Net-(P1-D-): track 9.67 -> 11.5 mm, vias 0 -> 1
